Commit message: Refactor material definitions in URDF files to comment out unused materials

File: XARM/demo/mbot_demo/urdf/mbot.urdf.xacro (robot description, xacro)
@@ -18,7 +18,7 @@
     <color rgba="1 0.4 0 1"/>
   </material>
-  <material name="black">
+  <!-- <material name="black">
     <color rgba="0 0 0 0.95"/>
-  </material>
+  </material> -->
   <material name="gray">
     <color rgba="0.75 0.75 0.75 1"/>
@@ -81,5 +81,5 @@
           <sphere radius="${caster_radius}" />
         </geometry>
-        <material name="black" />
+        <!-- <material name="black" /> -->
       </visual>
       <collision>

File: XARM/xarm_description/urdf/camera/camera.gazebo.xacro (robot description, xacro)
@@ -15,5 +15,5 @@
           <sphere radius="0.02"/>
         </geometry>
-        <material name="${prefix}White" />
+        <!-- <material name="${prefix}White" /> -->
       </visual>
       <collision>
@@ -30,5 +30,5 @@
     </joint>
     <gazebo reference="${prefix}link_camera">
-      <material>Gazebo/Black</material>
+      <!-- <material>Gazebo/Black</material> -->
     </gazebo>
     <gazebo reference="${prefix}link_camera">

File: XARM/xarm_description/urdf/common/common.link.xacro (robot description, xacro)
@@ -40,5 +40,4 @@
       </geometry>
       <origin xyz="${origin_xyz}" rpy="${origin_rpy}"/>
-      <material name="${material_name}" />
     </visual>
   </xacro:macro>

File: XARM/xarm_description/urdf/common/common.material.xacro (robot description, xacro)
@@ -2,5 +2,5 @@
 <robot xmlns:xacro="http://ros.org/wiki/xacro">
   <xacro:macro name="common_material" params="prefix">
-    <material name="${prefix}Black">
+    <!-- <material name="${prefix}Black">
       <color rgba="0.0 0.0 0.0 1.0"/>
     </material>
@@ -13,5 +13,5 @@
     <material name="${prefix}Silver">
       <color rgba="0.753 0.753 0.753 1.0"/>
-    </material>
+    </material> -->
   </xacro:macro>
 </robot>

File: XARM/xarm_description/urdf/other/other_geometry.urdf.xacro (robot description, xacro)
@@ -78,5 +78,5 @@
           </xacro:if>
         </geometry>
-        <material name="${prefix}White" />
+        <!-- <material name="${prefix}White" /> -->
       </visual>
       <collision>

File: XARM/xarm_description/urdf/xarm7/xarm7.urdf.xacro (robot description, xacro)
@@ -63,6 +63,5 @@
         mesh_filename="${visual_dir}/link_base"
         origin_xyz="0 0 0"
-        origin_rpy="0 0 0"
-        material_name="${prefix}White" />
+        origin_rpy="0 0 0" />
       <xacro:common_link_collision
         mesh_filename="${collision_dir}/link_base"
@@ -79,6 +78,5 @@
         mesh_filename="${visual_dir}/link1"
         origin_xyz="0 0 0"
-        origin_rpy="0 0 0"
-        material_name="${prefix}White" />
+        origin_rpy="0 0 0" />
       <xacro:common_link_collision
         mesh_filename="${collision_dir}/link1"
@@ -108,6 +106,5 @@
         mesh_filename="${visual_dir}/link2"
         origin_xyz="0 0 0"
-        origin_rpy="0 0 0"
-        material_name="${prefix}White" />
+        origin_rpy="0 0 0" />
       <xacro:common_link_collision
         mesh_filename="${collision_dir}/link2"
@@ -137,6 +134,5 @@
         mesh_filename="${visual_dir}/link3"
         origin_xyz="0 0 0"
-        origin_rpy="0 0 0"
-        material_name="${prefix}White" />
+        origin_rpy="0 0 0" />
       <xacro:common_link_collision
         mesh_filename="${collision_dir}/link3"
@@ -166,6 +162,5 @@
         mesh_filename="${visual_dir}/link4"
         origin_xyz="0 0 0"
-        origin_rpy="0 0 0"
-        material_name="${prefix}White" />
+        origin_rpy="0 0 0" />
       <xacro:common_link_collision
         mesh_filename="${collision_dir}/link4"
@@ -195,6 +190,5 @@
         mesh_filename="${visual_dir}/link5"
         origin_xyz="0 0 0"
-        origin_rpy="0 0 0"
-        material_name="${prefix}White" />
+        origin_rpy="0 0 0" />
       <xacro:common_link_collision
         mesh_filename="${collision_dir}/link5"
@@ -224,6 +218,5 @@
         mesh_filename="${visual_dir}/link6"
         origin_xyz="0 0 0"
-        origin_rpy="0 0 0"
-        material_name="${prefix}White" />
+        origin_rpy="0 0 0" />
       <xacro:common_link_collision
         mesh_filename="${collision_dir}/link6"
@@ -253,6 +246,5 @@
         mesh_filename="${link7_visual}"
         origin_xyz="0 0 0"
-        origin_rpy="0 0 0"
-        material_name="${prefix}Silver" />
+        origin_rpy="0 0 0" />
       <xacro:common_link_collision
         mesh_filename="${link7_collision}"

File: XARM/xarm_description/urdf/xarm7/xarm7_robot_macro.xacro (robot description, xacro)
@@ -5,4 +5,5 @@
     hw_ns:='xarm'
     limited:=false
+    is_ros2:=true
     velocity_control:=false
     add_gripper:=false

File: XARM/xarm_description/urdf/xarm_device.urdf.xacro (robot description, xacro)
@@ -34,5 +34,5 @@
   <xacro:arg name="baud_checkset" default="true"/>
   <xacro:arg name="default_gripper_baud" default="2000000"/>
-  <xacro:arg name="attach_to" default="world"/>
+  <xacro:arg name="attach_to" default="base_footprint"/>
   <xacro:arg name="attach_xyz" default="0 0 0"/>
   <xacro:arg name="attach_rpy" default="0 0 0"/>
