Commit message: Update URDF and SRDF configurations for NaviArm robot, adjusting file paths and mass properties

File: XARM/xarm_description/urdf/xarm7/xarm7.urdf.xacro (robot description, xacro)
@@ -55,5 +55,5 @@
       <inertial>
         <origin xyz="-0.021131 -0.0016302 0.056488" rpy="0 0 0" />
-        <mass value="0.88556" />
+        <mass value="0.3" />
         <inertia
           ixx="0.0030595" ixy="0.00012259" ixz="-0.00062705"

File: XARM/xarm_moveit_config/srdf/_xarm7_macro.srdf.xacro (robot description, xacro)
@@ -10,5 +10,5 @@
   <!-- SUBGROUPS: Groups can also be formed by referencing to already defined group names -->
   <xacro:macro name="xarm7_macro_srdf" params="prefix=''
-    add_gripper='false' add_vacuum_gripper='false' add_bio_gripper='false' add_other_geometry='false' ">
+    add_gripper='false' add_vacuum_gripper='true' add_bio_gripper='false' add_other_geometry='false' ">
     <group name="${prefix}xarm7">
       <joint name="${prefix}world_joint" />
