Commit message: Add Gazebo material definition for link_eef in realsense_d435i URDF

File: XARM/xarm_description/urdf/camera/realsense_d435i.urdf.xacro (robot description, xacro)
@@ -15,4 +15,7 @@
         origin_rpy="0 0 0" />
     </link>
+    <gazebo reference="${prefix}link_eef">
+      <material>Gazebo/Orange</material>
+    </gazebo>
     <xacro:if value="${add_d435i_links}">
       <link name="${prefix}camera_link"></link>
